File: ATtiny412 SOIC-8 Breakout PCB/ATtiny412 SOIC-8 Breakout PCB.kicad_pcb (KiCad board)
At the start: 2 copper layers, 25.4 x 20.3 mm, 11 parts, among them J1 Conn_01x03_Male, J2 Conn_01x04_Male, J3 Conn_01x04_Male, SW1 SW_MEC_5E, U1 MIC6315, U2 ATtiny412-SS

Commit message: Renamed files, minor fixes.
Corrected silk screen, and net names.
Other:
- board text added: "UPDI"
- board text removed: "PDI"
Changed lines of the file:
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@@
-(kicad_pcb (version 20171130) (host pcbnew "(5.1.9)-1")
+(kicad_pcb (version 20171130) (host pcbnew "(5.1.10)-1")
   (general
     (thickness 1.6)
@@
   )
   (page A4)
+  (title_block
+    (title "ATtiny412 SOIC-8 Breakout PCB")
+    (date 2021-08-21)
+    (rev B)
+  )
   (layers
     (0 F.Cu signal)
@@
   )
   (setup
-    (last_trace_width 0.254)
+    (last_trace_width 0.1524)
     (user_trace_width 0.254)
     (user_trace_width 0.508)
@@
     (add_net GND)
     (add_net "Net-(D1-Pad1)")
-    (add_net "Net-(SW1-Pad2)")
     (add_net VCC)
   )
@@
     (tags "resistor 0805")
     (attr smd)
-    (fp_text reference R2 (at 0 -1.7) (layer F.SilkS)
+    (fp_text reference R2 (at 0 -1.397) (layer F.SilkS)
       (effects (font (size 0.508 0.508) (thickness 0.0762)))
     )
@@
     (effects (font (size 0.508 0.508) (thickness 0.0762)))
   )
-  (gr_text PDI (at 140.208 91.44 90) (layer F.SilkS)
-    (effects (font (size 0.508 0.508) (thickness 0.0762)))
-  )
+  (gr_text UPDI (at 140.208 91.44 90) (layer F.SilkS)
+    (effects (font (size 0.508 0.508) (thickness 0.0762)))
+  )
